Commit message: got the robot to move, but using the wrong drive plugin lmao. made the middle wheels the drivers and made the other wheels frictionless to use diff_drive. DO NOT KEEP IT THIS WAY

File: description/gazebo_control.xacro (robot description, xacro)
@@ -2,4 +2,20 @@
 <robot xmlns:xacro="http://www.ros.org/wiki/xacro"  name="robot">
     <gazebo>
+        <plugin name="diff_drive" filename="libgazebo_ros_diff_drive.so">
+            <!-- Wheel Information -->
+            <left_joint>middle_left_wheel_joint</left_joint>
+            <right_joint>middle_right_wheel_joint</right_joint>
+            <wheel_separation>${chassis_y / 2}</wheel_separation>
+            <wheel_diameter>0.2</wheel_diameter>
+            <!-- Limits -->
+            <max_wheel_torque>20</max_wheel_torque>
+            <max_wheel_acceleration>10</max_wheel_acceleration>
+            <!-- Output -->
+            <odometry_frame>odom</odometry_frame>
+            <robot_base_frame>base_link</robot_base_frame>
+            <publish_odom>true</publish_odom>
+            <publish_odom_tf>true</publish_odom_tf>
+            <publish_wheel_tf>true</publish_wheel_tf>
+        </plugin>
     </gazebo>
 </robot>

File: description/robot_core.xacro (robot description, xacro)
@@ -46,5 +46,5 @@
         <parent link="base_link"/>
         <child link="front_left_wheel"/>
-        <origin xyz="${(wheel_radius * 2) + 0.045} ${chassis_y / 2} 0" rpy="-${pi / 2} 0 0"/>
+        <origin xyz="${wheel_radius + wheel_separation} ${chassis_y / 2} 0" rpy="-${pi / 2} 0 0"/>
         <axis xyz="0 0 1"/>
     </joint>
@@ -67,4 +67,6 @@
     <gazebo reference="front_left_wheel">
         <material>Gazebo/Blue</material>
+        <mu1 value="0"/>
+        <mu2 value="0"/>
     </gazebo>
     <!-- Middle Left Wheel Link -->
@@ -98,5 +100,5 @@
         <parent link="base_link"/>
         <child link="back_left_wheel"/>
-        <origin xyz="-${(wheel_radius * 2) + 0.045} ${chassis_y / 2} 0" rpy="-${pi / 2} 0 0"/>
+        <origin xyz="-${wheel_radius + wheel_separation} ${chassis_y / 2} 0" rpy="-${pi / 2} 0 0"/>
         <axis xyz="0 0 1"/>
     </joint>
@@ -119,4 +121,6 @@
     <gazebo reference="back_left_wheel">
         <material>Gazebo/Blue</material>
+        <mu1 value="0"/>
+        <mu2 value="0"/>
     </gazebo>
     <!-- Front Right Wheel Link -->
@@ -124,5 +128,5 @@
         <parent link="base_link"/>
         <child link="front_right_wheel"/>
-        <origin xyz="${(wheel_radius * 2) + 0.045} -${chassis_y / 2} 0" rpy="-${pi / 2} 0 ${pi}"/>
+        <origin xyz="${wheel_radius + wheel_separation} -${chassis_y / 2} 0" rpy="-${pi / 2} 0 ${pi}"/>
         <axis xyz="0 0 -1"/>
     </joint>
@@ -145,4 +149,6 @@
     <gazebo reference="front_right_wheel">
         <material>Gazebo/Blue</material>
+        <mu1 value="0"/>
+        <mu2 value="0"/>
     </gazebo>
     <!-- Middle Right Wheel Link -->
@@ -176,5 +182,5 @@
         <parent link="base_link"/>
         <child link="back_right_wheel"/>
-        <origin xyz="-${(wheel_radius * 2) + 0.045} -${chassis_y / 2} 0" rpy="-${pi / 2} 0 ${pi}"/>
+        <origin xyz="-${wheel_radius + wheel_separation} -${chassis_y / 2} 0" rpy="-${pi / 2} 0 ${pi}"/>
         <axis xyz="0 0 -1"/>
     </joint>
@@ -197,4 +203,6 @@
     <gazebo reference="back_right_wheel">
         <material>Gazebo/Blue</material>
+        <mu1 value="0"/>
+        <mu2 value="0"/>
     </gazebo>
 </robot>

File: description/robot_description.xacro (robot description, xacro)
@@ -1,8 +1,9 @@
 <?xml version="1.0"?>
 <robot xmlns:xacro="http://www.ros.org/wiki/xacro"  name="robot">
-    <xacro:property name="chassis_x" value="0.57"/>
+    <xacro:property name="chassis_x" value="0.568"/>
     <xacro:property name="chassis_y" value="0.4464"/>
     <xacro:property name="chassis_z" value="0.2632"/>
-    <xacro:property name="wheel_radius" value="0.08"/>
+    <xacro:property name="wheel_radius" value="0.1"/>
     <xacro:property name="wheel_length" value="0.09525"/>
+    <xacro:property name="wheel_separation" value="${(chassis_x - (wheel_radius * 2)) / 2}"/>
 </robot>
