Commit message: update refresh

File: description/depth_camera.xacro (robot description, xacro)
@@ -39,4 +39,8 @@
             </camera>
             <plugin name="camera_controller" filename="libgazebo_ros_camera.so">
+                <ros>
+                    <argument>~/out:=depthimage_to_laserscan</argument>
+                </ros>
+                <output_type>sensor_msgs/LaserScan</output_type>
                 <frame_name>camera_link_optical</frame_name>
                 <min_depth>0.1</min_depth>

File: description/robot_core.xacro (robot description, xacro)
@@ -16,4 +16,12 @@
     <!-- BASE LINK -->
     <link name="base_link">
+    </link>
+    <!-- BASE_FOOTPRINT LINK -->
+    <joint name="base_footprint_joint" type="fixed">
+        <parent link="base_link"/>
+        <child link="base_footprint"/>
+        <origin xyz="0 0 0" rpy="0 0 0"/>
+    </joint>
+    <link name="base_footprint">
     </link>
     <!-- CHASSIS LINK -->

Commit message: Added depth camera

File: description/depth_camera.xacro (robot description, xacro)
@@ -1,13 +1,14 @@
 <?xml version="1.0"?>
-<robot xmlns:xacro="http://www.ros.org/wiki/xacro" >
+<robot xmlns:xacro="http://www.ros.org/wiki/xacro"  name="robot">
+    <xacro:include filename="robot_description.xacro"/>
     <joint name="camera_joint" type="fixed">
         <parent link="chassis"/>
         <child link="camera_link"/>
-        <origin xyz="0.305 0 0.08" rpy="0 0 0"/>
+        <origin xyz="${chassis_x + 0.0125} 0 ${(chassis_z / 2)}" rpy="0 0 0"/>
     </joint>
     <link name="camera_link">
         <visual>
             <geometry>
-                <box size="0.010 0.03 0.03"/>
+                <box size="0.025 0.075 0.075"/>
             </geometry>
             <material name="red"/>
@@ -19,5 +20,5 @@
         <origin xyz="0 0 0" rpy="${-pi/2} 0 ${-pi/2}"/>
     </joint>
-    <link name="camera_link_optical"></link>
+    <link name="camera_link_optical"> </link>
     <gazebo reference="camera_link">
         <material>Gazebo/Red</material>
@@ -29,5 +30,5 @@
                 <horizontal_fov>1.089</horizontal_fov>
                 <image>
-                    <format>B8G8R8</format>
+                    <format>R8G8B8</format>
                     <width>640</width>
                     <height>480</height>
@@ -39,11 +40,5 @@
             </camera>
             <plugin name="camera_controller" filename="libgazebo_ros_camera.so">
-                <ros>
-                    <argument>~/out:=depthimage_to_laserscan</argument>
-                </ros>
-                <output_type>sensor_msgs/LaserScan</output_type>
                 <frame_name>camera_link_optical</frame_name>
-                <min_depth>0.1</min_depth>
-                <max_depth>100.0</max_depth>
             </plugin>
         </sensor>

File: description/robot.urdf.xacro (robot description, xacro)
@@ -4,4 +4,5 @@
     <xacro:include filename="gazebo_control.xacro"/>
     <xacro:include filename="lidar.xacro"/>
+    <xacro:include filename="depth_camera.xacro"/>
     <!--<xacro:include filename="urdf_rover.xacro"/> -->
     <!-- <xacro:include filename="urdf_arm.xacro"/> -->
