Commit message: Added the lidar to the urdf

File: description/robot.urdf.xacro (robot description, xacro)
@@ -4,3 +4,4 @@
     <xacro:include filename="gazebo_control.xacro"/>
     <xacro:include filename="depth_camera.xacro" />
+    <xacro:include filename="lidar.xacro"/>
 </robot>

File: description/robot_core.xacro (robot description, xacro)
@@ -13,4 +13,7 @@
     <material name="black">
         <color rgba="0 0 0 1" />
+    </material>
+    <material name="red">
+        <color rgba="1 0 0 1" />
     </material>
     <!-- BASE LINK -->

Commit message: idk

File: description/robot.urdf.xacro (robot description, xacro)
@@ -1,9 +1,9 @@
 <?xml version="1.0"?>
 <robot xmlns:xacro="http://www.ros.org/wiki/xacro"  name="robot">
-    <xacro:include filename="robot_core.xacro"/>
+   <xacro:include filename="robot_core.xacro"/>
     <xacro:include filename="gazebo_control.xacro"/>
     <xacro:include filename="lidar.xacro"/>
     <xacro:include filename="depth_camera.xacro"/>
-    <!--<xacro:include filename="urdf_rover.xacro"/> -->
+    <!--<xacro:include filename="urdf_rover.xacro"/>-->
     <!-- <xacro:include filename="urdf_arm.xacro"/> -->
 </robot>

File: description/urdf_rover.xacro (robot description, xacro)
@@ -4,59 +4,68 @@
      For more information, please see http://wiki.ros.org/sw_urdf_exporter -->
 <robot xmlns:xacro="http://www.ros.org/wiki/xacro"  name="robot">
-  <link
-  name="chassis">
-    <inertial>
-      <origin
-        xyz="0.0043448 0.25289 0.11566"
-        rpy="0 0 0" />
-      <mass
-        value="9.8064" />
-      <inertia
-        ixx="0.12153"
-        ixy="-0.00010062"
-        ixz="0.00012704"
-        iyy="0.16639"
-        iyz="-0.00019303"
-        izz="0.06694" />
-    </inertial>
-    <visual>
-      <origin
-        xyz="0 0 0"
-        rpy="0 0 0" />
-      <geometry>
-        <mesh
-          filename="package://billee_bot/meshes/chassis.STL" />
-      </geometry>
-      <material
-        name="">
-        <color
-          rgba="0.75294 0.75294 0.75294 1" />
-      </material>
-    </visual>
-    <collision>
-      <origin
-        xyz="0 0 0"
-        rpy="0 0 0" />
-      <geometry>
-        <mesh
-          filename="package://billee_bot/meshes/chassis.STL" />
-      </geometry>
-    </collision>
-  </link>
-  <link
-    name="differential">
-    <inertial>
-      <origin
-        xyz="-3.1443E-08 -0.019904 -2.4837E-08"
-        rpy="0 0 0" />
-      <mass
-        value="0.66325" />
-      <inertia
-        ixx="0.0053356"
-        ixy="1.0794E-10"
-        ixz="1.7412E-12"
-        iyy="0.0053078"
-        iyz="-2.6457E-10"
-        izz="0.00017607" />
+  <link name="base_link">
+  </link>
+  <joint name="origin_joint" type="fixed">
+    <parent link="base_link"/>
+    <child link="origin"/>
+    <origin xyz="0 0 2.5" rpy="0 0 0"/>
+  </joint>
+  <link
+    name="origin">
+    <inertial>
+      <origin
+        xyz="8.38288575652309E-07 0.131802961451061 0.119457737645149"
+        rpy="0 0 0" />
+      <mass
+        value="6.31210414331163" />
+      <inertia
+        ixx="0.109718503078251"
+        ixy="-3.107004482999E-07"
+        ixz="1.27742625490502E-09"
+        iyy="0.0504994066686463"
+        iyz="1.92825387800283E-10"
+        izz="0.157184029088834" />
+    </inertial>
+    <visual>
+      <origin
+        xyz="0 0 0"
+        rpy="0 0 0" />
+      <geometry>
+        <mesh
+          filename="package://billee_bot/meshes/origin.STL" />
+      </geometry>
+      <material
+        name="">
+        <color
+          rgba="0.752941176470588 0.752941176470588 0.752941176470588 1" />
+      </material>
+    </visual>
+    <collision>
+      <origin
+        xyz="0 0 0"
+        rpy="0 0 0" />
+      <geometry>
+        <mesh
+          filename="package://billee_bot/meshes/origin.STL" />
+      </geometry>
+    </collision>
+  </link>
+  <gazebo reference="origin">
+  </gazebo>
+  <link
+    name="differential_link">
+    <inertial>
+      <origin
+        xyz="2.48368055802417E-08 -3.14429672888805E-08 0.0199042487071119"
+        rpy="0 0 0" />
+      <mass
+        value="0.663253070147783" />
+      <inertia
+        ixx="0.000176065807329218"
+        ixy="-1.74124228174769E-12"
+        ixz="-2.64568230296014E-10"
+        iyy="0.00533562068145632"
+        iyz="-1.07943588779656E-10"
+        izz="0.00530780669766808" />
     </inertial>
     <visual>
@@ -71,5 +80,5 @@
         name="">
         <color
-          rgba="0.75294 0.75294 0.75294 1" />
+          rgba="0.752941176470588 0.752941176470588 0.752941176470588 1" />
       </material>
     </visual>
@@ -84,175 +93,179 @@
     </collision>
   </link>
-  <joint
-    name="differential"
-    type="continuous">
-    <origin
-      xyz="0 -0.013248 0.19342"
-      rpy="-1.5708 0 -1.5708" />
-    <parent
-      link="chassis" />
-    <child
-      link="differential" />
+  <gazebo reference="differential_link">
+  </gazebo>
+  <joint
+    name="differential_joint"
+    type="continuous">
+    <origin
+      xyz="0 0.0132475000000002 0.193421177067123"
+      rpy="0 0 0" />
+    <parent
+      link="origin" />
+    <child
+      link="differential_link" />
+    <axis
+      xyz="0 0 -1" />
+  </joint>
+  <link
+    name="xz_left">
+    <inertial>
+      <origin
+        xyz="-4.64889271523106E-09 0.0353830314295401 0.0108129499116387"
+        rpy="0 0 0" />
+      <mass
+        value="0.0155401592452895" />
+      <inertia
+        ixx="4.23350176895727E-06"
+        ixy="3.64217998809471E-14"
+        ixz="-3.64374435199193E-13"
+        iyy="5.22956405101389E-07"
+        iyz="1.47618341469402E-15"
+        izz="4.40773318106849E-06" />
+    </inertial>
+    <visual>
+      <origin
+        xyz="0 0 0"
+        rpy="0 0 0" />
+      <geometry>
+        <mesh
+          filename="package://billee_bot/meshes/xz_left.STL" />
+      </geometry>
+      <material
+        name="">
+        <color
+          rgba="0.752941176470588 0.752941176470588 0.752941176470588 1" />
+      </material>
+    </visual>
+    <collision>
+      <origin
+        xyz="0 0 0"
+        rpy="0 0 0" />
+      <geometry>
+        <mesh
+          filename="package://billee_bot/meshes/xz_left.STL" />
+      </geometry>
+    </collision>
+  </link>
+  <joint
+    name="link3_left"
+    type="continuous">
+    <origin
+      xyz="-0.248132600000003 0 0.00886587323959548"
+      rpy="0 0 0" />
+    <parent
+      link="differential_link" />
+    <child
+      link="xz_left" />
+    <axis
+      xyz="0 0 -1" />
+  </joint>
+  <gazebo reference="xz_left">
+  </gazebo>
+  <link
+    name="xy_left">
+    <inertial>
+      <origin
+        xyz="4.88970574419323E-05 0.0478926853579212 -1.29911378876635E-09"
+        rpy="0 0 0" />
+      <mass
+        value="0.0251600949304728" />
+      <inertia
+        ixx="1.39101472176527E-05"
+        ixy="-9.21531915994836E-11"
+        ixz="7.27350532600888E-12"
+        iyy="3.13190614602218E-06"
+        iyz="-7.09291132933723E-13"
+        izz="1.5415172628415E-05" />
+    </inertial>
+    <visual>
+      <origin
+        xyz="0 0 0"
+        rpy="0 0 0" />
+      <geometry>
+        <mesh
+          filename="package://billee_bot/meshes/xy_left.STL" />
+      </geometry>
+      <material
+        name="">
+        <color
+          rgba="0.752941176470588 0.752941176470588 0.752941176470588 1" />
+      </material>
+    </visual>
+    <collision>
+      <origin
+        xyz="0 0 0"
+        rpy="0 0 0" />
+      <geometry>
+        <mesh
+          filename="package://billee_bot/meshes/xy_left.STL" />
+      </geometry>
+    </collision>
+  </link>
+  <joint
+    name="link4_left"
+    type="continuous">
+    <origin
+      xyz="0 0.057190625 0.0108129496932786"
+      rpy="0 0 0" />
+    <parent
+      link="xz_left" />
+    <child
+      link="xy_left" />
     <axis
       xyz="0 1 0" />
   </joint>
   <link
-    name="xz_left">
-    <inertial>
-      <origin
-        xyz="-4.6489E-09 -0.035383 -0.010813"
-        rpy="0 0 0" />
-      <mass
-        value="0.01554" />
-      <inertia
-        ixx="4.2335E-06"
-        ixy="-3.6422E-14"
-        ixz="3.6437E-13"
-        iyy="5.2296E-07"
-        iyz="1.4762E-15"
-        izz="4.4077E-06" />
-    </inertial>
-    <visual>
-      <origin
-        xyz="0 0 0"
-        rpy="0 0 0" />
-      <geometry>
-        <mesh
-          filename="package://billee_bot/meshes/xz_left.STL" />
-      </geometry>
-      <material
-        name="">
-        <color
-          rgba="0.75294 0.75294 0.75294 1" />
-      </material>
-    </visual>
-    <collision>
-      <origin
-        xyz="0 0 0"
-        rpy="0 0 0" />
-      <geometry>
-        <mesh
-          filename="package://billee_bot/meshes/xz_left.STL" />
-      </geometry>
-    </collision>
-  </link>
-  <joint
-    name="link3_left"
-    type="continuous">
-    <origin
-      xyz="0 -0.0088659 0.24813"
-      rpy="1.5708 1.5708 0" />
-    <parent
-      link="differential" />
-    <child
-      link="xz_left" />
-    <axis
-      xyz="0 0 1" />
-  </joint>
-  <link
-    name="xy_left">
-    <inertial>
-      <origin
-        xyz="-4.8897E-05 0.047893 1.2991E-09"
-        rpy="0 0 0" />
-      <mass
-        value="0.02516" />
-      <inertia
-        ixx="1.391E-05"
-        ixy="9.2153E-11"
-        ixz="7.2735E-12"
-        iyy="3.1319E-06"
-        iyz="7.0929E-13"
-        izz="1.5415E-05" />
-    </inertial>
-    <visual>
-      <origin
-        xyz="0 0 0"
-        rpy="0 0 0" />
-      <geometry>
-        <mesh
-          filename="package://billee_bot/meshes/xy_left.STL" />
-      </geometry>
-      <material
-        name="">
-        <color
-          rgba="0.75294 0.75294 0.75294 1" />
-      </material>
-    </visual>
-    <collision>
-      <origin
-        xyz="0 0 0"
-        rpy="0 0 0" />
-      <geometry>
-        <mesh
-          filename="package://billee_bot/meshes/xy_left.STL" />
-      </geometry>
-    </collision>
-  </link>
-  <joint
-    name="link4_left"
-    type="continuous">
-    <origin
-      xyz="0 -0.057191 -0.010813"
-      rpy="0 0 3.1416" />
-    <parent
-      link="xz_left" />
-    <child
+    name="moment_left">
+    <inertial>
+      <origin
+        xyz="-0.0931762739376563 -0.123516160160037 -0.29938621188847"
+        rpy="0 0 0" />
+      <mass
+        value="2.01112856146357" />
+      <inertia
+        ixx="0.00516957821369544"
+        ixy="-0.000177768861031969"
+        ixz="-0.00023860509115917"
+        iyy="0.00729857222045286"
+        iyz="-0.00092981195043092"
+        izz="0.00746428128106379" />
+    </inertial>
+    <visual>
+      <origin
+        xyz="0 0 0"
+        rpy="0 0 0" />
+      <geometry>
+        <mesh
+          filename="package://billee_bot/meshes/moment_left.STL" />
+      </geometry>
+      <material
+        name="">
+        <color
+          rgba="0.752941176470588 0.752941176470588 0.752941176470588 1" />
+      </material>
+    </visual>
+    <collision>
+      <origin
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