Commit message: hehe

File: description/robot_values.xacro (robot description, xacro)
@@ -4,5 +4,5 @@
     <xacro:property name="chassis_y" value="0.4464"/>
     <xacro:property name="chassis_z" value="0.2632"/>
-    <xacro:property name="wheel_radius" value="0.1"/>
+    <xacro:property name="wheel_radius" value="0.1016"/>
     <xacro:property name="wheel_length" value="0.09525"/>
     <xacro:property name="wheel_separation" value="${(chassis_x - (wheel_radius * 2)) / 2}"/>

File: description/urdf_rover.xacro (robot description, xacro)
@@ -4,10 +4,13 @@
      For more information, please see http://wiki.ros.org/sw_urdf_exporter -->
 <robot xmlns:xacro="http://www.ros.org/wiki/xacro"  name="robot">
+  <xacro:include filename="robot_values.xacro"/>
   <link name="base_link">
   </link>
+  <gazebo reference="base_link">
+  </gazebo>
   <joint name="origin_joint" type="fixed">
     <parent link="base_link"/>
     <child link="origin"/>
-    <origin xyz="0 0 2.5" rpy="0 0 0"/>
+    <origin xyz="0 0 0.35" rpy="0 0 0"/>
   </joint>
   <link
@@ -33,19 +36,18 @@
       <geometry>
         <mesh
-          filename="package://billee_bot/meshes/origin.STL"/>
-      </geometry>
-      <material
-        name="">
-        <color
-          rgba="0.752941176470588 0.752941176470588 0.752941176470588 1" />
-      </material>
-    </visual>
-    <collision>
-      <origin
-        xyz="0 0 0"
-        rpy="0 0 0" />
-      <geometry>
-        <mesh
-          filename="package://billee_bot/meshes/origin.STL" />
+          filename="file://$(find billee_bot)/meshes/origin.STL"/>
+      </geometry>
+      <material
+        name="">
+        <color
+          rgba="0.752941176470588 0.752941176470588 0.752941176470588 1" />
+      </material>
+    </visual>
+    <collision>
+      <origin
+        xyz="0 ${(chassis_y / 2) - 0.08} ${chassis_z / 2}"
+        rpy="0 0 ${pi / 2}" />
+      <geometry>
+        <box size="${chassis_x} ${chassis_y} ${chassis_z}"/>
       </geometry>
     </collision>
@@ -75,19 +77,19 @@
       <geometry>
         <mesh
-          filename="package://billee_bot/meshes/differential.STL" />
-      </geometry>
-      <material
-        name="">
-        <color
-          rgba="0.752941176470588 0.752941176470588 0.752941176470588 1" />
-      </material>
-    </visual>
-    <collision>
-      <origin
-        xyz="0 0 0"
-        rpy="0 0 0" />
-      <geometry>
-        <mesh
-          filename="package://billee_bot/meshes/differential.STL" />
+          filename="file://$(find billee_bot)/meshes/differential.STL" />
+      </geometry>
+      <material
+        name="">
+        <color
+          rgba="0.752941176470588 0.752941176470588 0.752941176470588 1" />
+      </material>
+    </visual>
+    <collision>
+      <origin
+        xyz="0 0 0"
+        rpy="0 0 0" />
+      <geometry>
+        <mesh
+          filename="file://$(find billee_bot)/meshes/differential.STL" />
       </geometry>
     </collision>
@@ -96,6 +98,5 @@
   </gazebo>
   <joint
-    name="differential_joint"
-    type="continuous">
+    name="differential_joint" type="revolute">
     <origin
       xyz="0 0.0132475000000002 0.193421177067123"
@@ -106,5 +107,6 @@
       link="differential_link" />
     <axis
-      xyz="0 0 -1" />
+      xyz="0 0 1" />
+    <limit effort="100" lower="-${pi / 4}" upper="${pi / 4}" velocity="0"/>
   </joint>
   <link
@@ -130,19 +132,19 @@
       <geometry>
         <mesh
-          filename="package://billee_bot/meshes/xz_left.STL" />
-      </geometry>
-      <material
-        name="">
-        <color
-          rgba="0.752941176470588 0.752941176470588 0.752941176470588 1" />
-      </material>
-    </visual>
-    <collision>
-      <origin
-        xyz="0 0 0"
-        rpy="0 0 0" />
-      <geometry>
-        <mesh
-          filename="package://billee_bot/meshes/xz_left.STL" />
+          filename="file://$(find billee_bot)/meshes/xz_left.STL" />
+      </geometry>
+      <material
+        name="">
+        <color
+          rgba="0.752941176470588 0.752941176470588 0.752941176470588 1" />
+      </material>
+    </visual>
+    <collision>
+      <origin
+        xyz="0 0 0"
+        rpy="0 0 0" />
+      <geometry>
+        <mesh
+          filename="file://$(find billee_bot)/meshes/xz_left.STL" />
       </geometry>
     </collision>
@@ -185,19 +187,19 @@
       <geometry>
         <mesh
-          filename="package://billee_bot/meshes/xy_left.STL" />
-      </geometry>
-      <material
-        name="">
-        <color
-          rgba="0.752941176470588 0.752941176470588 0.752941176470588 1" />
-      </material>
-    </visual>
-    <collision>
-      <origin
-        xyz="0 0 0"
-        rpy="0 0 0" />
-      <geometry>
-        <mesh
-          filename="package://billee_bot/meshes/xy_left.STL" />
+          filename="file://$(find billee_bot)/meshes/xy_left.STL" />
+      </geometry>
+      <material
+        name="">
+        <color
+          rgba="0.752941176470588 0.752941176470588 0.752941176470588 1" />
+      </material>
+    </visual>
+    <collision>
+      <origin
+        xyz="0 0 0"
+        rpy="0 0 0" />
+      <geometry>
+        <mesh
+          filename="file://$(find billee_bot)/meshes/xy_left.STL" />
       </geometry>
     </collision>
@@ -238,19 +240,19 @@
       <geometry>
         <mesh
-          filename="package://billee_bot/meshes/moment_left.STL" />
-      </geometry>
-      <material
-        name="">
-        <color
-          rgba="0.752941176470588 0.752941176470588 0.752941176470588 1" />
-      </material>
-    </visual>
-    <collision>
-      <origin
-        xyz="0 0 0"
-        rpy="0 0 0" />
-      <geometry>
-        <mesh
-          filename="package://billee_bot/meshes/moment_left.STL" />
+          filename="file://$(find billee_bot)/meshes/moment_left.STL" />
+      </geometry>
+      <material
+        name="">
+        <color
+          rgba="0.752941176470588 0.752941176470588 0.752941176470588 1" />
+      </material>
+    </visual>
+    <collision>
+      <origin
+        xyz="0 0 0"
+        rpy="0 0 0" />
+      <geometry>
+        <mesh
+          filename="file://$(find billee_bot)/meshes/moment_left.STL" />
       </geometry>
     </collision>
@@ -258,8 +260,8 @@
   <joint
     name="link5_left"
-    type="continuous">
+    type="fixed">
     <origin
       xyz="0 0.05 0"
-      rpy="0 0 0" />
+      rpy="0.1 0 0" />
     <parent
       link="xy_left" />
@@ -291,19 +293,19 @@
       <geometry>
         <mesh
-          filename="package://billee_bot/meshes/v_sus_left.STL" />
-      </geometry>
-      <material
-        name="">
-        <color
-          rgba="0.752941176470588 0.752941176470588 0.752941176470588 1" />
-      </material>
-    </visual>
-    <collision>
-      <origin
-        xyz="0 0 0"
-        rpy="0 0 0" />
-      <geometry>
-        <mesh
-          filename="package://billee_bot/meshes/v_sus_left.STL" />
+          filename="file://$(find billee_bot)/meshes/v_sus_left.STL" />
+      </geometry>
+      <material
+        name="">
+        <color
+          rgba="0.752941176470588 0.752941176470588 0.752941176470588 1" />
+      </material>
+    </visual>
+    <collision>
+      <origin
+        xyz="0 0 0"
+        rpy="0 0 0" />
+      <geometry>
+        <mesh
+          filename="file://$(find billee_bot)/meshes/v_sus_left.STL" />
       </geometry>
     </collision>
@@ -344,19 +346,18 @@
       <geometry>
         <mesh
-          filename="package://billee_bot/meshes/back_wheel_left.STL" />
-      </geometry>
-      <material
-        name="">
-        <color
-          rgba="0.752941176470588 0.752941176470588 0.752941176470588 1" />
-      </material>
-    </visual>
-    <collision>
-      <origin
-        xyz="0 0 0"
-        rpy="0 0 0" />
-      <geometry>
-        <mesh
-          filename="package://billee_bot/meshes/back_wheel_left.STL" />
+          filename="file://$(find billee_bot)/meshes/back_wheel_left.STL" />
+      </geometry>
+      <material
+        name="">
+        <color
+          rgba="0.752941176470588 0.752941176470588 0.752941176470588 1" />
+      </material>
+    </visual>
+    <collision>
+      <origin
+        xyz="-${wheel_length / 2} 0 0"
+        rpy="0 -${pi / 2} 0" />
+      <geometry>
+        <cylinder radius="${wheel_radius}" length="${wheel_length}"/>
       </geometry>
     </collision>
@@ -379,4 +380,5 @@
       effort="0"
       velocity="0" />
+    <dynamics damping="0.4"/>
   </joint>
   <link
@@ -402,19 +404,18 @@
       <geometry>
         <mesh
-          filename="package://billee_bot/meshes/mid_wheel_left.STL" />
-      </geometry>
-      <material
-        name="">
-        <color
-          rgba="0.752941176470588 0.752941176470588 0.752941176470588 1" />
-      </material>
-    </visual>
-    <collision>
-      <origin
-        xyz="0 0 0"
-        rpy="0 0 0" />
-      <geometry>
-        <mesh
-          filename="package://billee_bot/meshes/mid_wheel_left.STL" />
+          filename="file://$(find billee_bot)/meshes/mid_wheel_left.STL" />
+      </geometry>
+      <material
+        name="">
+        <color
+          rgba="0.752941176470588 0.752941176470588 0.752941176470588 1" />
+      </material>
+    </visual>
+    <collision>
+      <origin
+        xyz="-${wheel_length / 2} 0 0"
+        rpy="0 -${pi / 2} 0" />
+      <geometry>
+        <cylinder radius="${wheel_radius}" length="${wheel_length}"/>
       </geometry>
     </collision>
@@ -437,4 +438,5 @@
       effort="0"
       velocity="0" />
+    <dynamics damping="0.4"/>
   </joint>
   <link
@@ -460,19 +462,18 @@
       <geometry>
         <mesh
-          filename="package://billee_bot/meshes/front_wheel_left.STL" />
-      </geometry>
-      <material
-        name="">
-        <color
-          rgba="0.752941176470588 0.752941176470588 0.752941176470588 1" />
-      </material>
-    </visual>
-    <collision>
-      <origin
-        xyz="0 0 0"
-        rpy="0 0 0" />
-      <geometry>
-        <mesh
-          filename="package://billee_bot/meshes/front_wheel_left.STL" />
+          filename="file://$(find billee_bot)/meshes/front_wheel_left.STL" />
+      </geometry>
+      <material
+        name="">
+        <color
+          rgba="0.752941176470588 0.752941176470588 0.752941176470588 1" />
+      </material>
+    </visual>
+    <collision>
+      <origin
+        xyz="-${wheel_length / 2} 0 0"
+        rpy="0 -${pi / 2} 0" />
+      <geometry>
+        <cylinder radius="${wheel_radius}" length="${wheel_length}"/>
       </geometry>
     </collision>
@@ -495,4 +496,5 @@
       effort="0"
       velocity="0" />
+    <dynamics damping="0.4"/>
   </joint>
   <link
@@ -518,19 +520,19 @@
       <geometry>
         <mesh
-          filename="package://billee_bot/meshes/xz_right.STL" />
-      </geometry>
-      <material
-        name="">
-        <color
-          rgba="0.752941176470588 0.752941176470588 0.752941176470588 1" />
-      </material>
-    </visual>
-    <collision>
-      <origin
-        xyz="0 0 0"
-        rpy="0 0 0" />
-      <geometry>
-        <mesh
-          filename="package://billee_bot/meshes/xz_right.STL" />
+          filename="file://$(find billee_bot)/meshes/xz_right.STL" />
+      </geometry>
+      <material
+        name="">
+        <color
+          rgba="0.752941176470588 0.752941176470588 0.752941176470588 1" />
+      </material>
+    </visual>
+    <collision>
+      <origin
+        xyz="0 0 0"
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